File: SchematicsAndInfo/ESP8266_YM2612_SN76489_VGM_Player/ESP8266_YM2612_SN76489_VGM_Player.sch (KiCad schematic (older format))
At the start: 46 parts, among them J1 STEREO_AUDIO_JACK, U1 NodeMCU_1.0_ESP8266, U10 PIC16F690-I/P, U11 LTC6903, U2 LM386, U3 LM386, U4 YM2612, U5 SN769486, U6 74HC595, U7 74HC595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

Commit message: Removed music.h include and corrected schematic label.
Parts:
- U5: value SN769486 -> SN76486
Changed lines of the file:
@@
 LIBS:nodemcu
 LIBS:ym2612
-LIBS:sn769486
-LIBS:SN74HC595_W_VCC
 LIBS:microchip_pic16mcu
 LIBS:ESP8266_YM2612_SN76489_VGM_Player-cache
@@
 P 6200 3850
 F 0 "U5" H 6250 4650 60  0000 C CNN
-F 1 "SN769486" H 6150 3550 60  0000 C CNN
+F 1 "SN76486" H 6150 3550 60  0000 C CNN
 F 2 "" H 6150 3550 60  0001 C CNN
 F 3 "" H 6150 3550 60  0001 C CNN

Commit message: Corrected schematic
Parts:
- U5: value SN76486 -> SN76489
Changed lines of the file:
@@
 P 6200 3850
 F 0 "U5" H 6250 4650 60  0000 C CNN
-F 1 "SN76486" H 6150 3550 60  0000 C CNN
+F 1 "SN76489" H 6150 3550 60  0000 C CNN
 F 2 "" H 6150 3550 60  0001 C CNN
 F 3 "" H 6150 3550 60  0001 C CNN
